File: stm32.kicad_sch (KiCad schematic)
At the start: 16 parts, among them J2 Conn_ARM_SWD_TagConnect_TC203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, Q1 2N7002, SW13 SW_Push, U3 STM32F072CBTx

Commit message: Add stm crystal, update title block, add power on LED for 3V3 line
Parts:
- added C8, C9: 18pF, Capacitor_SMD:C_0603_1608Metric, symbol Device:C_Small
- added D20: LED RED, LED_SMD:LED_0603_1608Metric, symbol Device:LED
- added R2: 100R, Resistor_SMD:R_0603_1608Metric, symbol Device:R_Small
- added Y1: 8MHz, Crystal:Crystal_SMD_Abracon_ABM3B-4Pin_5.0x3.2mm, symbol Device:Crystal_GND24
Connections:
- net 3V3: now also D20.2 (A)
- net GND: now also C8.2, C9.1, R2.1, Y1.2, Y1.4
- net OSC_IN: now also C8.1, Y1.1
- net OSC_OUT: now also C9.2, Y1.3
- new net: D20.1 (K), R2.2
Other:
- note added: "3V3 Power"
- company: (none) -> MadMan
- title: (none) -> Crumb Catcher

Commit message: Cleanup, Add usb emc and esd
Parts:
- renumbered R2 to R4, R2 to R5, R2 to R6, R2 to R7, U3 to U1

Commit message: Update BOM, start to fill in part metadata
Parts:
- C3, C4, C5, C6, C7: footprint Capacitor_SMD:C_0603_1608Metric -> Capacitor_SMD:C_0402_1005Metric; MPN (none) -> C0402C104K3RAC7867 KEMET $0.33 CAP CER 0.1UF 25V X7R 0402 D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; Manufacturer (none) -> KEMET; Price (none) -> $0.33; Rating (none) -> CAP CER 0.1UF 25V X7R 0402; Supplier (none) -> Digikey; Supplier PN (none) -> 399-14148-1-ND
- C8, C9: footprint Capacitor_SMD:C_0603_1608Metric -> Capacitor_SMD:C_0402_1005Metric; Digikey PN 311-3889-1-ND -> (none); MPN CC0603FRNPO9BN180 -> CC0402FRNPO9BN180; Notes CAP CER 18PF 50V C0G/NPO 0603 -> (none); Price (none) -> $0.16; Rating (none) -> CAP CER 18PF 50V C0G/NPO 0402; Supplier (none) -> Digikey; Supplier PN (none) -> 311-1643-1-ND
- D20: Digikey PN 732-4978-1-ND -> (none); Notes Red 625nm LED Indication - Discrete 2V 0603 (1608 Metric) -> (none); Price (none) -> $0.24; Rating (none) -> LED RED CLEAR 0603 SMD; Supplier (none) -> Digikey; Supplier PN (none) -> 732-4978-1-ND
- Y1: footprint Crystal:Crystal_SMD_Abracon_ABM3B-4Pin_5.0x3.2mm -> LocalLib:Crystal_SMD_ECX-32-4Pin_3.2x2.5mm; Digikey PN 535-9720-1-ND -> (none); MPN ABM3B-8.000MHZ-B2-T -> ECS-80-12-33-JGN-TR; Manufacturer Abracon LLC -> ECS Inc.; Notes CRYSTAL 8.0000MHZ 18PF SMD -> (none); Price (none) -> $1.00; Rating (none) -> CRYSTAL 8.0000MHZ 12PF SMD; Supplier (none) -> Digikey; Supplier PN (none) -> 50-ECS-80-12-33-JGN-CT-ND
