File: Switches.kicad_sch (KiCad schematic)
At the start: 30 parts, among them SW10 SW_SPST, SW11 PEC11R, SW2 PEC11R, SW3 SW_SPST, SW4 SW_SPST, SW5 PEC11R, SW6 SW_SPST, SW7 SW_SPST, SW9 SW_SPST

Commit message: Update BOM,
Parts:
- C10: renamed from C20; MPN C0402C104K3RAC7867 -> CC0402KPX7R9BB104; Manufacturer KEMET -> YAGEO; Price $0.33 -> $0.17; Rating CAP CER 0.1UF 25V X7R 0402 -> CAP 0402 50V 100 NF X7R; Supplier PN 399-14148-1-ND -> 13-CC0402KPX7R9BB104CT-ND
- C11: renamed from C21; MPN C0402C104K3RAC7867 -> CC0402KPX7R9BB104; Manufacturer KEMET -> YAGEO; Price $0.33 -> $0.17; Rating CAP CER 0.1UF 25V X7R 0402 -> CAP 0402 50V 100 NF X7R; Supplier PN 399-14148-1-ND -> 13-CC0402KPX7R9BB104CT-ND
- C6: renamed from C28; MPN C0402C104K3RAC7867 -> CC0402KPX7R9BB104; Manufacturer KEMET -> YAGEO; Price $0.33 -> $0.17; Rating CAP CER 0.1UF 25V X7R 0402 -> CAP 0402 50V 100 NF X7R; Supplier PN 399-14148-1-ND -> 13-CC0402KPX7R9BB104CT-ND
- C7: renamed from C29; MPN C0402C104K3RAC7867 -> CC0402KPX7R9BB104; Manufacturer KEMET -> YAGEO; Price $0.33 -> $0.17; Rating CAP CER 0.1UF 25V X7R 0402 -> CAP 0402 50V 100 NF X7R; Supplier PN 399-14148-1-ND -> 13-CC0402KPX7R9BB104CT-ND
- C8: renamed from C26; MPN C0402C104K3RAC7867 -> CC0402KPX7R9BB104; Manufacturer KEMET -> YAGEO; Price $0.33 -> $0.17; Rating CAP CER 0.1UF 25V X7R 0402 -> CAP 0402 50V 100 NF X7R; Supplier PN 399-14148-1-ND -> 13-CC0402KPX7R9BB104CT-ND
- C9: renamed from C27; MPN C0402C104K3RAC7867 -> CC0402KPX7R9BB104; Manufacturer KEMET -> YAGEO; Price $0.33 -> $0.17; Rating CAP CER 0.1UF 25V X7R 0402 -> CAP 0402 50V 100 NF X7R; Supplier PN 399-14148-1-ND -> 13-CC0402KPX7R9BB104CT-ND
- D10: renamed from D12; value WS2812C-2020 -> SK6812_MINI_E; MPN (none) -> SK6812MINI-E; Price (none) -> $0.44; Rating (none) -> 3.7...5.3V; Supplier (none) -> LCSC; Supplier PN (none) -> C5149201
- D11: renamed from D15; value WS2812C-2020 -> SK6812_MINI_E; MPN (none) -> SK6812MINI-E; Price (none) -> $0.44; Rating (none) -> 3.7...5.3V; Supplier (none) -> LCSC; Supplier PN (none) -> C5149201
- D15: renamed from D13; value WS2812C-2020 -> SK6812_MINI_E; MPN (none) -> SK6812MINI-E; Price (none) -> $0.44; Rating (none) -> 3.7...5.3V; Supplier (none) -> LCSC; Supplier PN (none) -> C5149201
- D16: value WS2812C-2020 -> SK6812_MINI_E; MPN (none) -> SK6812MINI-E; Price (none) -> $0.44; Rating (none) -> 3.7...5.3V; Supplier (none) -> LCSC; Supplier PN (none) -> C5149201
- D5: renamed from D11; value WS2812C-2020 -> SK6812_MINI_E; MPN (none) -> SK6812MINI-E; MPN  WS2812C-2020 -> SK6812_MINI_E; Price (none) -> $0.44; Rating (none) -> 3.7...5.3V; Supplier (none) -> LCSC; Supplier PN (none) -> C5149201
- D6: renamed from D14; value WS2812C-2020 -> SK6812_MINI_E; MPN (none) -> SK6812MINI-E; Price (none) -> $0.44; Rating (none) -> 3.7...5.3V; Supplier (none) -> LCSC; Supplier PN (none) -> C5149201
- renumbered D5 to D12, D9 to D13, D10 to D14, D8 to D17, D2 to D7, D6 to D8, D7 to D9, SW2 to SW1, SW3 to SW2, SW4 to SW3, SW5 to SW4, SW6 to SW5, SW7 to SW6, SW11 to SW7, SW9 to SW8, SW10 to SW9
Other:
- moved on the sheet: C10, C11, C6, C7, C8, C9, D10, D11, D12, D13, D14, D15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

Commit message: Clear ERC's
Parts:
- renumbered C6 to C19, C7 to C20, C8 to C21, C9 to C22, C10 to C23, C11 to C24, D17 to D18, SW9 to SW10, SW1 to SW2, SW2 to SW3, SW3 to SW4, SW4 to SW5, SW5 to SW6, SW6 to SW7, SW7 to SW8, SW8 to SW9
Changed lines of the file:
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@@
 		(dnp no)
 		(fields_autoplaced yes)
-		(property "Reference" "C6"
+		(property "Reference" "C19"
 			(at 80.01 29.8512 0)
 			(effects
@@
 			(project "CrumbCatcherLight"
 				(path "/eedae293-eb5b-47bd-b383-bccfdf81bf72/1682b9f6-7d62-400a-a0b2-d2d916d42f36"
-					(reference "C6")
+					(reference "C19")
 					(unit 1)
 				)
@@
 		(dnp no)
 		(fields_autoplaced yes)
-		(property "Reference" "SW5"
+		(property "Reference" "SW6"
 			(at 149.86 82.55 0)
 			(effects
@@
 			(project "CrumbCatcherLight"
 				(path "/eedae293-eb5b-47bd-b383-bccfdf81bf72/1682b9f6-7d62-400a-a0b2-d2d916d42f36"
-					(reference "SW5")
+					(reference "SW6")
 					(unit 1)
 				)
@@
 		(dnp no)
 		(fields_autoplaced yes)
-		(property "Reference" "C9"
+		(property "Reference" "C22"
 			(at 130.81 34.9312 0)
 			(effects
@@
 			(project "CrumbCatcherLight"
 				(path "/eedae293-eb5b-47bd-b383-bccfdf81bf72/1682b9f6-7d62-400a-a0b2-d2d916d42f36"
-					(reference "C9")
+					(reference "C22")
 					(unit 1)
 				)
@@
 		(on_board yes)
 		(dnp no)
-		(property "Reference" "SW1"
+		(property "Reference" "SW2"
 			(at 94.996 27.305 0)
 			(effects
@@
 			(project "CrumbCatcherLight"
 				(path "/eedae293-eb5b-47bd-b383-bccfdf81bf72/1682b9f6-7d62-400a-a0b2-d2d916d42f36"
-					(reference "SW1")
+					(reference "SW2")
 					(unit 1)
 				)
@@
 		(dnp no)
 		(fields_autoplaced yes)
-		(property "Reference" "SW2"
+		(property "Reference" "SW3"
 			(at 99.06 57.15 0)
 			(effects
@@
 			(project "CrumbCatcherLight"
 				(path "/eedae293-eb5b-47bd-b383-bccfdf81bf72/1682b9f6-7d62-400a-a0b2-d2d916d42f36"
-					(reference "SW2")
+					(reference "SW3")
 					(unit 1)
 				)
@@
 		(dnp no)
 		(fields_autoplaced yes)
-		(property "Reference" "SW8"
+		(property "Reference" "SW9"
 			(at 204.47 57.15 0)
 			(effects
@@
 			(project "CrumbCatcherLight"
 				(path "/eedae293-eb5b-47bd-b383-bccfdf81bf72/1682b9f6-7d62-400a-a0b2-d2d916d42f36"
-					(reference "SW8")
+					(reference "SW9")
 					(unit 1)
 				)
@@
 		(on_board yes)
 		(dnp no)
-		(property "Reference" "SW4"
+		(property "Reference" "SW5"
 			(at 145.796 27.305 0)
 			(effects
@@
 			(project "CrumbCatcherLight"
 				(path "/eedae293-eb5b-47bd-b383-bccfdf81bf72/1682b9f6-7d62-400a-a0b2-d2d916d42f36"
-					(reference "SW4")
+					(reference "SW5")
 					(unit 1)
 				)
@@
 		(dnp no)
 		(fields_autoplaced yes)
-		(property "Reference" "C7"
+		(property "Reference" "C20"
 			(at 80.01 34.9312 0)
 			(effects
@@
 			(project "CrumbCatcherLight"
 				(path "/eedae293-eb5b-47bd-b383-bccfdf81bf72/1682b9f6-7d62-400a-a0b2-d2d916d42f36"
-					(reference "C7")
+					(reference "C20")
 					(unit 1)
 				)
@@
 		(dnp no)
 		(fields_autoplaced yes)
-		(property "Reference" "SW3"
+		(property "Reference" "SW4"
 			(at 99.06 82.55 0)
 			(effects
@@
 			(project "CrumbCatcherLight"
 				(path "/eedae293-eb5b-47bd-b383-bccfdf81bf72/1682b9f6-7d62-400a-a0b2-d2d916d42f36"
-					(reference "SW3")
+					(reference "SW4")
 					(unit 1)
 				)
@@
 		(on_board yes)
 		(dnp no)
-		(property "Reference" "SW7"
+		(property "Reference" "SW8"
 			(at 200.406 27.305 0)
 			(effects
@@
 			(project "CrumbCatcherLight"
 				(path "/eedae293-eb5b-47bd-b383-bccfdf81bf72/1682b9f6-7d62-400a-a0b2-d2d916d42f36"
-					(reference "SW7")
+					(reference "SW8")
 					(unit 1)
 				)
@@
 		(dnp no)
 		(fields_autoplaced yes)
-		(property "Reference" "SW9"
+		(property "Reference" "SW10"
 			(at 204.47 82.55 0)
 			(effects
@@
 			(project "CrumbCatcherLight"
 				(path "/eedae293-eb5b-47bd-b383-bccfdf81bf72/1682b9f6-7d62-400a-a0b2-d2d916d42f36"
-					(reference "SW9")
+					(reference "SW10")
 					(unit 1)
 				)
@@
 		(dnp no)
 		(fields_autoplaced yes)
-		(property "Reference" "C8"
+		(property "Reference" "C21"
 			(at 130.81 29.8512 0)
 			(effects
@@
 			(project "CrumbCatcherLight"
 				(path "/eedae293-eb5b-47bd-b383-bccfdf81bf72/1682b9f6-7d62-400a-a0b2-d2d916d42f36"
-					(reference "C8")
+					(reference "C21")
 					(unit 1)
 				)
@@
 		(dnp no)
 		(fields_autoplaced yes)
-		(property "Reference" "C11"
+		(property "Reference" "C24"
 			(at 185.42 34.9312 0)
 			(effects
@@
 			(project "CrumbCatcherLight"
 				(path "/eedae293-eb5b-47bd-b383-bccfdf81bf72/1682b9f6-7d62-400a-a0b2-d2d916d42f36"
-					(reference "C11")
+					(reference "C24")
 					(unit 1)
 				)
@@
 		(dnp no)
 		(fields_autoplaced yes)
-		(property "Reference" "SW6"
+		(property "Reference" "SW7"
 			(at 153.67 57.15 0)
 			(effects
@@
 			(project "CrumbCatcherLight"
 				(path "/eedae293-eb5b-47bd-b383-bccfdf81bf72/1682b9f6-7d62-400a-a0b2-d2d916d42f36"
-					(reference "SW6")
+					(reference "SW7")
 					(unit 1)
 				)
@@
 		(dnp no)
 		(fields_autoplaced yes)
-		(property "Reference" "C10"
+		(property "Reference" "C23"
 			(at 185.42 29.8512 0)
 			(effects
@@
 			(project "CrumbCatcherLight"
 				(path "/eedae293-eb5b-47bd-b383-bccfdf81bf72/1682b9f6-7d62-400a-a0b2-d2d916d42f36"
-					(reference "C10")
+					(reference "C23")
 					(unit 1)
 				)
@@
 		(dnp no)
 		(fields_autoplaced yes)
-		(property "Reference" "D17"
+		(property "Reference" "D18"
 			(at 207.01 42.5449 90)
 			(effects
@@
 			(project "CrumbCatcherLight"
 				(path "/eedae293-eb5b-47bd-b383-bccfdf81bf72/1682b9f6-7d62-400a-a0b2-d2d916d42f36"
-					(reference "D17")
+					(reference "D18")
 					(unit 1)
 				)

Commit message: Update to nRF52840 module, add BQ for battery charging
Parts:
- D10, D11, D15, D16, D6: MPN  WS2812C-2020 -> (none); Manufacturer Worldsemi -> Worldsemi; Supplier PN C5149201 -> C5149201
- D12, D13, D14, D18, D3, D4, D7, D8, D9: Price $0.18 -> $0.18
- D5: MPN  SK6812_MINI_E -> (none); Manufacturer Worldsemi -> Worldsemi; Supplier PN C5149201 -> C5149201
- SW2, SW5, SW8: Price $3.37 -> $3.37
Changed lines of the file:
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@@
 			)
 		)
-		(property "MPN " "SK6812_MINI_E"
+		(property "Manufacturer" "Worldsemi"
 			(at 95.885 113.665 0)
 			(effects
@@
 			)
 		)
-		(property "Manufacturer" "Worldsemi "
+		(property "JLC Basic" "N"
 			(at 95.885 113.665 0)
 			(effects
@@
 			)
 		)
-		(property "JLC Basic" "N"
+		(property "Substitute" "N"
 			(at 95.885 113.665 0)
 			(effects
@@
 			)
 		)
-		(property "Substitute" "N"
+		(property "Price" "$0.44"
 			(at 95.885 113.665 0)
 			(effects
@@
 			)
 		)
-		(property "Price" "$0.44"
+		(property "Interface" ""
 			(at 95.885 113.665 0)
 			(effects
@@
 			)
 		)
-		(property "Interface" ""
+		(property "Rating" " 3.7...5.3V"
 			(at 95.885 113.665 0)
 			(effects
@@
 			)
 		)
-		(property "Rating" " 3.7...5.3V"
+		(property "Supplier" "LCSC"
 			(at 95.885 113.665 0)
 			(effects
@@
 			)
 		)
-		(property "Supplier" "LCSC"
+		(property "Supplier PN" "C5149201"
 			(at 95.885 113.665 0)
 			(effects
@@
 			)
 		)
-		(property "Supplier PN" "C5149201 "
+		(property "MPN" "SK6812MINI-E"
 			(at 95.885 113.665 0)
 			(effects
@@
 			)
 		)
-		(property "MPN" "SK6812MINI-E"
+		(property "Config" ""
+			(at 95.885 113.665 0)
+			(effects
+				(font
+					(size 1.27 1.27)
+				)
+				(hide yes)
+			)
+		)
+		(property "digikey" ""
+			(at 95.885 113.665 0)
+			(effects
+				(font
+					(size 1.27 1.27)
+				)
+				(hide yes)
+			)
+		)
+		(property "mouser" ""
 			(at 95.885 113.665 0)
 			(effects
@@
 		)
 		(instances
-			(project "CrumbCatcherLight"
+			(project ""
+				(path "/eedae293-eb5b-47bd-b383-bccfdf81bf72"
+					(reference "D5")
+					(unit 1)
+				)
 				(path "/eedae293-eb5b-47bd-b383-bccfdf81bf72/1682b9f6-7d62-400a-a0b2-d2d916d42f36"
 					(reference "D5")
@@
 			)
 		)
-		(property "Price" "$0.18 "
+		(property "Price" "$0.18"
 			(at 90.17 63.5 0)
 			(effects
@@
 			)
 		)
-		(property "Price" "$0.18 "
+		(property "Price" "$0.18"
 			(at 90.17 88.9 0)
 			(effects
@@
 			)
 		)
-		(property "Price" "$3.37 "
+		(property "Price" "$3.37"
 			(at 95.25 33.655 0)
 			(effects
@@
 			)
 		)
-		(property "Price" "$0.18 "
+		(property "Price" "$0.18"
 			(at 195.58 88.9 0)
 			(effects
@@
 			)
 		)
-		(property "MPN " "WS2812C-2020"
-			(at 197.485 132.715 0)
-			(effects
-				(font
-					(size 1.27 1.27)
-				)
-				(hide yes)
-			)
-		)
-		(property "Manufacturer" "Worldsemi "
+		(property "Manufacturer" "Worldsemi"
 			(at 197.485 132.715 0)
 			(effects
@@
 			)
 		)
-		(property "Supplier PN" "C5149201 "
+		(property "Supplier PN" "C5149201"
 			(at 197.485 132.715 0)
 			(effects
@@
 			)
 		)
-		(property "MPN " "WS2812C-2020"
-			(at 146.685 113.665 0)
-			(effects
-				(font
-					(size 1.27 1.27)
-				)
-				(hide yes)
-			)
-		)
-		(property "Manufacturer" "Worldsemi "
+		(property "Manufacturer" "Worldsemi"
 			(at 146.685 113.665 0)
 			(effects
@@
 			)
 		)
-		(property "Supplier PN" "C5149201 "
+		(property "Supplier PN" "C5149201"
 			(at 146.685 113.665 0)
 			(effects
@@
 			)
 		)
-		(property "MPN " "WS2812C-2020"
-			(at 146.685 132.715 0)
-			(effects
-				(font
-					(size 1.27 1.27)
-				)
-				(hide yes)
-			)
-		)
-		(property "Manufacturer" "Worldsemi "
+		(property "Manufacturer" "Worldsemi"
 			(at 146.685 132.715 0)
 			(effects
@@
 			)
 		)
-		(property "Supplier PN" "C5149201 "
+		(property "Supplier PN" "C5149201"
 			(at 146.685 132.715 0)
 			(effects
@@
 			)
 		)
-		(property "Price" "$3.37 "
+		(property "Price" "$3.37"
 			(at 146.05 33.655 0)
 			(effects
@@
 			)
 		)
-		(property "Price" "$0.18 "
+		(property "Price" "$0.18"
 			(at 104.14 43.815 0)
 			(effects
@@
 			)
 		)
-		(property "MPN " "WS2812C-2020"
-			(at 95.885 132.715 0)
-			(effects
-				(font
-					(size 1.27 1.27)
-				)
-				(hide yes)
-			)
-		)
-		(property "Manufacturer" "Worldsemi "
+		(property "Manufacturer" "Worldsemi"
 			(at 95.885 132.715 0)
 			(effects
@@
 			)
 		)
-		(property "Supplier PN" "C5149201 "
+		(property "Supplier PN" "C5149201"
 			(at 95.885 132.715 0)
 			(effects
@@
 			)
 		)
-		(property "Price" "$0.18 "
+		(property "Price" "$0.18"
 			(at 195.58 63.5 0)
 			(effects
@@
 			)
 		)
-		(property "Price" "$0.18 "
+		(property "Price" "$0.18"
 			(at 140.97 88.9 0)
 			(effects
@@
 			)
 		)
-		(property "Price" "$0.18 "
+		(property "Price" "$0.18"
 			(at 154.94 43.815 0)
 			(effects
@@
 			)
 		)
-		(property "Price" "$3.37 "
+		(property "Price" "$3.37"
 			(at 200.66 33.655 0)
 			(effects
@@
 			)
 		)
-		(property "MPN " "WS2812C-2020"
-			(at 197.485 113.665 0)
-			(effects
-				(font
-					(size 1.27 1.27)
-				)
-				(hide yes)
-			)
-		)
-		(property "Manufacturer" "Worldsemi "
+		(property "Manufacturer" "Worldsemi"
 			(at 197.485 113.665 0)
 			(effects
@@
 			)
 		)
-		(property "Supplier PN" "C5149201 "
+		(property "Supplier PN" "C5149201"
 			(at 197.485 113.665 0)
 			(effects
@@
 			)
 		)
-		(property "Price" "$0.18 "
+		(property "Price" "$0.18"
 			(at 140.97 63.5 0)
 			(effects
@@
 			)
 		)
-		(property "Price" "$0.18 "
+		(property "Price" "$0.18"
 			(at 209.55 43.815 0)
 			(effects

Commit message: Add some todo notes, add 3/2 pin battery connectors
Add NTC connector, Update power scheme for RF module
Parts:
- renumbered C19 to C4, C20 to C5, C21 to C6, C22 to C7, C23 to C8, C24 to C9, D18 to D17, SW2 to SW1, SW3 to SW2, SW4 to SW3, SW5 to SW4, SW6 to SW5, SW7 to SW6, SW8 to SW7, SW9 to SW8, SW10 to SW9
Changed lines of the file:
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@@
 		(dnp no)
 		(fields_autoplaced yes)
-		(property "Reference" "C19"
+		(property "Reference" "C4"
 			(at 80.01 29.8512 0)
 			(effects
@@
 			(project "CrumbCatcherLight"
 				(path "/eedae293-eb5b-47bd-b383-bccfdf81bf72/1682b9f6-7d62-400a-a0b2-d2d916d42f36"
-					(reference "C19")
+					(reference "C4")
 					(unit 1)
 				)
@@
 		(dnp no)
 		(fields_autoplaced yes)
-		(property "Reference" "SW6"
+		(property "Reference" "SW5"
 			(at 149.86 82.55 0)
 			(effects
@@
 			(project "CrumbCatcherLight"
 				(path "/eedae293-eb5b-47bd-b383-bccfdf81bf72/1682b9f6-7d62-400a-a0b2-d2d916d42f36"
-					(reference "SW6")
+					(reference "SW5")
 					(unit 1)
 				)
@@
 		(dnp no)
 		(fields_autoplaced yes)
-		(property "Reference" "C22"
+		(property "Reference" "C7"
 			(at 130.81 34.9312 0)
 			(effects
@@
 			(project "CrumbCatcherLight"
 				(path "/eedae293-eb5b-47bd-b383-bccfdf81bf72/1682b9f6-7d62-400a-a0b2-d2d916d42f36"
-					(reference "C22")
+					(reference "C7")
 					(unit 1)
 				)
@@
 		(on_board yes)
 		(dnp no)
-		(property "Reference" "SW2"
+		(property "Reference" "SW1"
 			(at 94.996 27.305 0)
 			(effects
@@
 			(project "CrumbCatcherLight"
 				(path "/eedae293-eb5b-47bd-b383-bccfdf81bf72/1682b9f6-7d62-400a-a0b2-d2d916d42f36"
-					(reference "SW2")
+					(reference "SW1")
 					(unit 1)
 				)
@@
 		(dnp no)
 		(fields_autoplaced yes)
-		(property "Reference" "SW3"
+		(property "Reference" "SW2"
 			(at 99.06 57.15 0)
 			(effects
@@
 			(project "CrumbCatcherLight"
 				(path "/eedae293-eb5b-47bd-b383-bccfdf81bf72/1682b9f6-7d62-400a-a0b2-d2d916d42f36"
-					(reference "SW3")
+					(reference "SW2")
 					(unit 1)
 				)
@@
 		(dnp no)
 		(fields_autoplaced yes)
-		(property "Reference" "SW9"
+		(property "Reference" "SW8"
 			(at 204.47 57.15 0)
 			(effects
@@
 			(project "CrumbCatcherLight"
 				(path "/eedae293-eb5b-47bd-b383-bccfdf81bf72/1682b9f6-7d62-400a-a0b2-d2d916d42f36"
-					(reference "SW9")
+					(reference "SW8")
 					(unit 1)
 				)
@@
 		(on_board yes)
 		(dnp no)
-		(property "Reference" "SW5"
+		(property "Reference" "SW4"
 			(at 145.796 27.305 0)
 			(effects
@@
 			(project "CrumbCatcherLight"
 				(path "/eedae293-eb5b-47bd-b383-bccfdf81bf72/1682b9f6-7d62-400a-a0b2-d2d916d42f36"
-					(reference "SW5")
+					(reference "SW4")
 					(unit 1)
 				)
@@
 		(dnp no)
 		(fields_autoplaced yes)
-		(property "Reference" "C20"
+		(property "Reference" "C5"
 			(at 80.01 34.9312 0)
 			(effects
@@
 			(project "CrumbCatcherLight"
 				(path "/eedae293-eb5b-47bd-b383-bccfdf81bf72/1682b9f6-7d62-400a-a0b2-d2d916d42f36"
-					(reference "C20")
+					(reference "C5")
 					(unit 1)
 				)
@@
 		(dnp no)
 		(fields_autoplaced yes)
-		(property "Reference" "SW4"
+		(property "Reference" "SW3"
 			(at 99.06 82.55 0)
 			(effects
@@
 			(project "CrumbCatcherLight"
 				(path "/eedae293-eb5b-47bd-b383-bccfdf81bf72/1682b9f6-7d62-400a-a0b2-d2d916d42f36"
-					(reference "SW4")
+					(reference "SW3")
 					(unit 1)
 				)
@@
 		(on_board yes)
 		(dnp no)
-		(property "Reference" "SW8"
+		(property "Reference" "SW7"
 			(at 200.406 27.305 0)
 			(effects
@@
 			(project "CrumbCatcherLight"
 				(path "/eedae293-eb5b-47bd-b383-bccfdf81bf72/1682b9f6-7d62-400a-a0b2-d2d916d42f36"
-					(reference "SW8")
+					(reference "SW7")
 					(unit 1)
 				)
@@
 		(dnp no)
 		(fields_autoplaced yes)
-		(property "Reference" "SW10"
+		(property "Reference" "SW9"
 			(at 204.47 82.55 0)
 			(effects
@@
 			(project "CrumbCatcherLight"
 				(path "/eedae293-eb5b-47bd-b383-bccfdf81bf72/1682b9f6-7d62-400a-a0b2-d2d916d42f36"
-					(reference "SW10")
+					(reference "SW9")
 					(unit 1)
 				)
@@
 		(dnp no)
 		(fields_autoplaced yes)
-		(property "Reference" "C21"
+		(property "Reference" "C6"
 			(at 130.81 29.8512 0)
 			(effects
@@
 			(project "CrumbCatcherLight"
 				(path "/eedae293-eb5b-47bd-b383-bccfdf81bf72/1682b9f6-7d62-400a-a0b2-d2d916d42f36"
-					(reference "C21")
+					(reference "C6")
 					(unit 1)
 				)
@@
 		(dnp no)
 		(fields_autoplaced yes)
-		(property "Reference" "C24"
+		(property "Reference" "C9"
 			(at 185.42 34.9312 0)
 			(effects
@@
 			(project "CrumbCatcherLight"
 				(path "/eedae293-eb5b-47bd-b383-bccfdf81bf72/1682b9f6-7d62-400a-a0b2-d2d916d42f36"
-					(reference "C24")
+					(reference "C9")
 					(unit 1)
 				)
@@
 		(dnp no)
 		(fields_autoplaced yes)
-		(property "Reference" "SW7"
+		(property "Reference" "SW6"
 			(at 153.67 57.15 0)
 			(effects
@@
 			(project "CrumbCatcherLight"
 				(path "/eedae293-eb5b-47bd-b383-bccfdf81bf72/1682b9f6-7d62-400a-a0b2-d2d916d42f36"
-					(reference "SW7")
+					(reference "SW6")
 					(unit 1)
 				)
@@
 		(dnp no)
 		(fields_autoplaced yes)
-		(property "Reference" "C23"
+		(property "Reference" "C8"
 			(at 185.42 29.8512 0)
 			(effects
@@
 			(project "CrumbCatcherLight"
 				(path "/eedae293-eb5b-47bd-b383-bccfdf81bf72/1682b9f6-7d62-400a-a0b2-d2d916d42f36"
-					(reference "C23")
+					(reference "C8")
 					(unit 1)
 				)
@@
 		(dnp no)
 		(fields_autoplaced yes)
-		(property "Reference" "D18"
+		(property "Reference" "D17"
 			(at 207.01 42.5449 90)
 			(effects
@@
 			(project "CrumbCatcherLight"
 				(path "/eedae293-eb5b-47bd-b383-bccfdf81bf72/1682b9f6-7d62-400a-a0b2-d2d916d42f36"
-					(reference "D18")
+					(reference "D17")
 					(unit 1)
 				)

Commit message: Update BOM
Parts:
- removed C9: 100nF, Capacitor_SMD:C_0402_1005Metric, symbol Device:C_Small
- added C12: 100nF, Capacitor_SMD:C_0603_1608Metric, symbol Device:C_Small
- C4, C5, C6, C7, C8: footprint Capacitor_SMD:C_0402_1005Metric -> Capacitor_SMD:C_0603_1608Metric; LCSC (none) -> C432917; MPN CC0402KPX7R9BB104 -> CC0603KPX7R9BB104; Price $0.17 -> $0.10; Rating CAP 0402 50V 100 NF X7R -> CAP CER 0.1UF 50V X7R 0603; Supplier PN 13-CC0402KPX7R9BB104CT-ND -> (none); digikey (none) -> 311-3567-1-ND; mouser (none) -> 603-CC603KPX7R9BB104
Connections:
- net ENC1A: now also C5.1; no longer C4.1
- net ENC1B: now also C4.2; no longer C5.2
- net ENC2A: now also C7.1; no longer C6.1
- net ENC2B: now also C6.2; no longer C7.2
- net ENC3A: now also C12.1; no longer C8.1
- net ENC3B: now also C8.2
- net GND: now also C4.1, C5.2, C6.1, C7.2, C8.1, C12.2; no longer C4.2, C5.1, C6.2, C7.1, C8.2
Other:
- moved on the sheet: D10, D11, D12, D15, D16, D17, D5, D6, D7, SW1, SW4, SW7
