File: nRF52840.kicad_sch (KiCad schematic)
At the start: 5 parts, among them U2 nRF52840, U6 NCP1117-3.3

Commit message: Update to nRF52840 module, add BQ for battery charging
Parts:
- removed C27, C28, C29: 10uF, Capacitor_SMD:C_0805_2012Metric, symbol Device:C_Small
- removed U2: nRF52840, Package_DFN_QFN:Nordic_AQFN-73-1EP_7x7mm_P0.5mm, symbol MCU_Nordic:nRF52840
- removed U6: NCP1117-3.3, Package_TO_SOT_SMD:SOT-223-3_TabPin2, symbol Regulator_Linear:NCP1117-3.3_SOT223
- added C30, C31: 8pF, Capacitor_SMD:C_0603_1608Metric, symbol Device:C_Small
- added C32: 1uF, Capacitor_SMD:C_0603_1608Metric, symbol Device:C_Small
- added C33: 100nF, Capacitor_SMD:C_0603_1608Metric, symbol Device:C_Small
- added C34, C35: 4.7uF, Capacitor_SMD:C_0805_2012Metric, symbol Device:C_Small
- added D19: Yellow, LED_SMD:LED_0603_1608Metric, symbol Device:LED_Small
- added D20: GREEN, LED_SMD:LED_0603_1608Metric, symbol Device:LED_Small
- added J3: Conn_ARM_SWD_TagConnect_TC2030-NL, Connector:Tag-Connect_TC2030-IDC-NL_2x03_P1.27mm_Vertical, symbol Connector:Conn_ARM_SWD_TagConnect_TC2030-NL
- added JP1: Charge Boost, Jumper:SolderJumper-2_P1.3mm_Open_RoundedPad1.0x1.5mm, symbol Jumper:Jumper_2_Open
- added R13: 2M, Resistor_SMD:R_0603_1608Metric, symbol Device:R_Small
- added R14: 806k, Resistor_SMD:R_0603_1608Metric, symbol Device:R_Small
- added R17: 1K, Resistor_SMD:R_0402_1005Metric, symbol Device:R_Small
- added R18, R19, R23: 1K, Resistor_SMD:R_0603_1608Metric, symbol Device:R_Small
- added R20, R21, R22: 10K, Resistor_SMD:R_0603_1608Metric, symbol Device:R_Small
- added SW11: EVPAA202K, Mad_Footprints:EVP-AA202K, symbol Switch:SW_Push
- added U2: MDBT50Q-U1MV2, Mad_Footprints:Raytac_MDBT50Q, symbol Mad_Symbols:MDBT50Q-U1MV2
- added U6: BQ24075RGT, Package_DFN_QFN:VQFN-16-1EP_3x3mm_P0.5mm_EP1.6x1.6mm, symbol Battery_Management:BQ24075RGT
- added X2: 32.768kHz, symbol PCM_Crystal_AKL:Crystal_Generic
Connections:
- net 3V3: now also J3.1 (VCC)
- net GND: now also C30.2, C31.2, C32.1, C33.2, C34.2, C35.2, D20.1 (K), J3.5 (GND), R13.1, R19.1, R20.2, R21.1, R23.1, SW11.2, U2.1 (GND), U2.15 (GND), U2.2 (GND), U2.33 (GND), U2.55 (GND), U6.15 (SYSOFF), U6.17 (VSS), U6.4 (~{CE}), U6.5 (EN2), U6.8 (VSS)
- new net: R18.1, R19.2
- new net: JP1.2 (B), R18.2
- new net: D19.2 (A), R22.2
- new net: C31.1, U2.18 (P0.01/XL2), X2.1
- new net: C30.1, U2.17 (P0.00/XL1), X2.2
- new net: R21.2, U6.1 (TS)
- new net: D20.2 (A), R17.1
- new net: R23.2, U6.12 (ILIM)
- new net: JP1.1 (A), R20.1, U6.16 (ISET)
- new net: D19.1 (K), U6.9 (~{CHG})
- new net BLED: R17.2, U2.19 (P0.26)
- new net BVOLT: R13.2, R14.1, U2.20 (P0.04)
- new net COL0: U2.8 (P1.15)
- new net COL1: U2.10 (P0.29)
- new net COL10: U2.57 (P1.06)
- new net COL11: U2.59 (P1.05)
- new net COL12: U2.61 (P1.01)
- new net COL13: U2.50 (P1.02)
- new net COL2: U2.12 (P0.31)
- new net COL3: U2.14 (P0.30)
- new net COL4: U2.13 (P0.28)
- new net COL5: U2.11 (P0.02)
- new net COL6: U2.9 (P0.03)
- new net COL7: U2.60 (P1.03)
- new net COL8: U2.58 (P1.07)
- new net COL9: U2.56 (P1.04)
- new net NFC1: U2.52 (P0.09)
- new net NFC2: U2.54 (P0.10)
- new net P0.20: U2.44 (P0.20)
- new net P0.21: U2.43 (P0.21)
- new net P0.22: U2.46 (P0.22)
- new net P0.24: U2.48 (P0.24)
- new net P0.25: U2.49 (P0.25)
- new net POWER_PIN: U2.21 (P0.05)
- new net RGB: U2.16 (P0.27)
- new net ROW0: U2.7 (P1.14)
- new net ROW1: U2.6 (P1.13)
- new net ROW2: U2.5 (P1.12)
- new net ROW3: U2.4 (P1.11)
- new net ROW4: U2.3 (P1.10)
- new net SWCLK: J3.4 (SWCLK), U2.53 (SWDCLK)
- new net SWDIO: J3.2 (SWDIO), U2.51 (SWDIO)
- new net USB_D_N: U2.34 (D-)
- new net USB_D_P: U2.35 (D+)
- new net VBAT: C35.1, R14.2, U6.2 (BAT), U6.3 (BAT)
- new net VBUS: C32.2, C33.1, U2.32 (VBUS), U6.13 (IN)
- new net VDDH: C34.1, R22.1, U2.28 (VDD), U2.30 (VDDH), U6.10 (OUT), U6.11 (OUT), U6.6 (EN1)
- new net ~{RST}: J3.3 (~{RESET}), SW11.1, U2.40 (P0.18/~{RST})
- no-connect marks 0 -> 19
Other:
- note added: "BQ24075RGTR"
- note added: "MDBT50Q-U1MV2"
- note added: "Status LED"
- note added: "TAG Connect"
- note added: "TODO: Spec Crystal and Caps Properly"
- note added: "TODO: Spec Power Regulator, BVOLT voltage divider."
- note added: "Update"
- note added: "Work out what to connect VCC of the Tag Connect to"
- note removed: "3V3 Reg"

Commit message: More research, added connector for Qi charger in
Parts:
- removed C32: 1uF, Capacitor_SMD:C_0603_1608Metric, symbol Device:C_Small
- removed C33: 100nF, Capacitor_SMD:C_0603_1608Metric, symbol Device:C_Small
- removed C34, C35: 4.7uF, Capacitor_SMD:C_0805_2012Metric, symbol Device:C_Small
- removed D19: Yellow, LED_SMD:LED_0603_1608Metric, symbol Device:LED_Small
- removed JP1: Charge Boost, Jumper:SolderJumper-2_P1.3mm_Open_RoundedPad1.0x1.5mm, symbol Jumper:Jumper_2_Open
- removed R13: 2M, Resistor_SMD:R_0603_1608Metric, symbol Device:R_Small
- removed R14: 806k, Resistor_SMD:R_0603_1608Metric, symbol Device:R_Small
- removed R18, R19, R23: 1K, Resistor_SMD:R_0603_1608Metric, symbol Device:R_Small
- removed R20, R21, R22: 10K, Resistor_SMD:R_0603_1608Metric, symbol Device:R_Small
- removed U6: BQ24075RGT, Package_DFN_QFN:VQFN-16-1EP_3x3mm_P0.5mm_EP1.6x1.6mm, symbol Battery_Management:BQ24075RGT
Connections:
- net VDDH is gone; now on net 3V3: U2.28 (VDD), U2.30 (VDDH)
- no-connect marks 19 -> 17
Other:
- note added: "Confirm 3V3 is ok power in for this module"
- note removed: "BQ24075RGTR"
- note removed: "TODO: Spec Power Regulator, BVOLT voltage divider."
- moved on the sheet: C30, C31, SW11, U2, X2

Commit message: Add some todo notes, add 3/2 pin battery connectors
Add NTC connector, Update power scheme for RF module
Parts:
- removed C31: 8pF, Capacitor_SMD:C_0603_1608Metric, symbol Device:C_Small
- added C14, C15: 10uF, Capacitor_SMD:C_0805_2012Metric, symbol Device:C_Small
- added C17: 12pF, Capacitor_SMD:C_0603_1608Metric, symbol Device:C_Small
- added L1: 10uH, symbol Device:L_Small
- C16: renamed from C30; value 8pF -> 12pF; LCSC C432917 -> (none); MPN CC0603KPX7R9BB104 -> (none); Manufacturer YAGEO -> (none); Price $0.10 -> (none); Rating CAP CER 0.1UF 50V X7R 0603 -> (none); Supplier Digikey -> (none); digikey 311-3567-1-ND -> (none); mouser 603-CC603KPX7R9BB104 -> (none)
- renumbered D20 to D19, J3 to J6, R17 to R12, SW11 to SW10, U2 to U4, X2 to X1
Connections:
- net 3V3: no longer U4.28 (VDD), U4.30 (VDDH)
- net GND: now also C14.1, C15.1, C17.2
- net at U4.18 (P0.01/XL2), X1.1: now also C17.1
- net at U4.31 (DCCH): now also L1.2
- net VBUS renamed V_{IN}
- net V_{IN}: now also U4.30 (VDDH), C14.2
- new net: C15.2, L1.1, U4.28 (VDD)
- no-connect marks 17 -> 16
Other:
- note added: "Look into either running a DC/DC outside or running Module with DC/DC internal working."

Commit message: Update BOM
Parts:
- removed R12: 1K, Resistor_SMD:R_0402_1005Metric, symbol Device:R_Small
- added C18: 10uF, Capacitor_SMD:C_0805_2012Metric, symbol Device:C_Small
- added R13: 1K, Resistor_SMD:R_0603_1608Metric, symbol Device:R_Small
- C16, C17: MPN (none) -> CC0603FRNPO8BN120; Manufacturer (none) -> YAGEO; Price (none) -> $0.15; Rating (none) -> CAP CER 12PF 25V C0G/NPO 0603; Supplier (none) -> Digikey; digikey (none) -> 13-CC0603FRNPO8BN120CT-ND
- L1: footprint (none) -> Inductor_SMD:L_0603_1608Metric; MPN (none) -> CBMF1608T100K; Manufacturer (none) -> Taiyo Yuden; Price (none) -> $0.16; Rating (none) -> FIXED IND 10UH 380MA 468MOHM SMD; Supplier (none) -> Digikey; digikey (none) -> 587-1720-1-ND
- X1: footprint (none) -> Mad_Footprints:XTAL_FC-12M; MPN (none) -> FC-12M 32.7680KA-A3; Manufacturer (none) -> EPSON; Price (none) -> $1.35; Rating (none) -> CRYSTAL 32.7680KHZ 12.5PF SMD; Supplier (none) -> Digikey; digikey (none) -> SER3672CT-ND
Connections:
- net BLED: now also R13.2
- net GND: now also C18.1
- net at D19.2 (A): now also R13.1
- net V_{IN} renamed VDDH
- net VDDH: no longer U4.32 (VBUS)
- new net V_{BUS}: C18.2, U4.32 (VBUS)
Other:
- note removed: "Confirm 3V3 is ok power in for this module"
- note removed: "Look into either running a DC/DC outside or running Module with DC/DC internal working."
- note removed: "TODO: Spec Crystal and Caps Properly"
- note removed: "Update"
- title: (none) -> Crumb Catcher
- moved on the sheet: C14, D19

Commit message: Add some research, update switches
Parts:
- renumbered C16 to C10, C17 to C11, C14 to C7, C18 to C8, C15 to C9, D19 to D4, R13 to R12, SW10 to SW1
Changed lines of the file:
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@@
 		(dnp no)
 		(fields_autoplaced yes)
-		(property "Reference" "C18"
+		(property "Reference" "C8"
 			(at 204.47 74.9235 0)
 			(effects
@@
 			(project "CrumbCatcherLight"
 				(path "/eedae293-eb5b-47bd-b383-bccfdf81bf72/5668be87-7451-4e35-a0d8-99be4b22c9c7"
-					(reference "C18")
+					(reference "C8")
 					(unit 1)
 				)
@@
 		(on_board yes)
 		(dnp no)
-		(property "Reference" "R13"
+		(property "Reference" "R12"
 			(at 386.715 35.56 0)
 			(effects
@@
 			(project "CrumbCatcherLight"
 				(path "/eedae293-eb5b-47bd-b383-bccfdf81bf72/5668be87-7451-4e35-a0d8-99be4b22c9c7"
-					(reference "R13")
+					(reference "R12")
 					(unit 1)
 				)
@@
 		(dnp no)
 		(fields_autoplaced yes)
-		(property "Reference" "C15"
+		(property "Reference" "C9"
 			(at 231.14 78.7335 0)
 			(effects
@@
 			(project "CrumbCatcherLight"
 				(path "/eedae293-eb5b-47bd-b383-bccfdf81bf72/5668be87-7451-4e35-a0d8-99be4b22c9c7"
-					(reference "C15")
+					(reference "C9")
 					(unit 1)
 				)
@@
 		(on_board yes)
 		(dnp no)
-		(property "Reference" "C17"
+		(property "Reference" "C11"
 			(at 259.0863 110.49 90)
 			(effects
@@
 			(project "CrumbCatcherLight"
 				(path "/eedae293-eb5b-47bd-b383-bccfdf81bf72/5668be87-7451-4e35-a0d8-99be4b22c9c7"
-					(reference "C17")
+					(reference "C11")
 					(unit 1)
 				)
@@
 		(on_board yes)
 		(dnp no)
-		(property "Reference" "SW10"
+		(property "Reference" "SW1"
 			(at 254 130.81 0)
 			(effects
@@
 			(project "CrumbCatcherLight"
 				(path "/eedae293-eb5b-47bd-b383-bccfdf81bf72/5668be87-7451-4e35-a0d8-99be4b22c9c7"
-					(reference "SW10")
+					(reference "SW1")
 					(unit 1)
 				)
@@
 		(dnp no)
 		(fields_autoplaced yes)
-		(property "Reference" "C14"
+		(property "Reference" "C7"
 			(at 191.77 74.9235 0)
 			(effects
@@
 			(project "CrumbCatcherLight"
 				(path "/eedae293-eb5b-47bd-b383-bccfdf81bf72/5668be87-7451-4e35-a0d8-99be4b22c9c7"
-					(reference "C14")
+					(reference "C7")
 					(unit 1)
 				)
@@
 		(dnp no)
 		(fields_autoplaced yes)
-		(property "Reference" "C16"
+		(property "Reference" "C10"
 			(at 259.0863 82.55 90)
 			(effects
@@
 			(project ""
 				(path "/eedae293-eb5b-47bd-b383-bccfdf81bf72/5668be87-7451-4e35-a0d8-99be4b22c9c7"
-					(reference "C16")
+					(reference "C10")
 					(unit 1)
 				)
@@
 		(on_board yes)
 		(dnp no)
-		(property "Reference" "D19"
+		(property "Reference" "D4"
 			(at 390.525 41.275 90)
 			(effects
@@
 			(project "CrumbCatcherLight"
 				(path "/eedae293-eb5b-47bd-b383-bccfdf81bf72/5668be87-7451-4e35-a0d8-99be4b22c9c7"
-					(reference "D19")
+					(reference "D4")
 					(unit 1)
 				)
